File: PCB/DeskFighter/DeskFighter.kicad_sch (KiCad schematic)
At the start: 195 parts, among them SW1 1U, SW10 1U, SW11 1U, SW12 1U, SW13 1U, SW14 1U, SW15 1U, SW16 1U, SW17 1U, SW18 1U, SW19 1U, SW2 1U, SW20 1U, SW21 1U, SW22 1U, SW23 1U, SW24 1U, SW25 1U, SW26 1U, SW27 1U, SW28 1U, SW29 1U, SW3 1U, SW30 1U, SW31 1U, SW32 1U, SW33 1U, SW34 1U, SW35 1U, SW36 1U, SW37 1U, SW38 1U, SW39 1U, SW4 1U, SW40 1U, SW41 1U, SW42 1U, SW43 1U, SW44 1U, SW45 1U, SW46 1U, SW47 1U, SW48 1U, SW49 1U, SW5 1U, SW50 1U, SW51 1U, SW52 1U, SW53 1U, SW54 1U, SW55 1U, SW56 1U, SW57 1U, SW58 1U, SW59 1U, SW6 1U, SW60 1U, SW61 1U, SW62 1U, SW63 1U, SW64 1U, SW65 1U, SW66 2U, SW67 1U, SW68 1U, SW69 1U, SW7 1U, SW70 1U, SW71 1U, SW72 1U, SW73 1U, SW74 1U, SW75 1U, SW76 1U, SW77 1U, SW78 1U, SW79 1U, SW8 1U, SW80 1U, SW81 1U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

Commit message: Add more diodes, adjust num/caps label placement
Bump board version to 1.1
Ghosting was a problem with fast typing or button-mashing.
Parts:
- D28, D30, D45, D47, D61, D63, D74, D76, D85, D86, D87: value Placeholder -> 1N4148W; footprint DeskFighter:DiodePlaceholder -> DeskFighter:D_SOD-123_Handsolder; symbol DeskFighter:Diode_Placeholder -> Diode:1N4148W; now in the parts list
